Commit message: test gym

File: src/myur5e/myur5e_description/urdf/mybox.urdf.xacro (robot description, xacro)
@@ -3,10 +3,10 @@
     <link name="mybox">
         <inertial>
-            <origin xyz="2 0 0" />
+            <origin xyz="0 0 0" />
             <mass value="0.2" />
             <inertia  ixx="1.0" ixy="0.0"  ixz="0.0"  iyy="100.0"  iyz="0.0"  izz="1.0" />
         </inertial>
         <visual>
-            <origin xyz="2 0 1"/>
+            <origin xyz="0 0 0"/>
             <geometry>
                 <box size="0.05 0.05 0.05" />
@@ -14,5 +14,5 @@
         </visual>
         <collision>
-            <origin xyz="2 0 1"/>
+            <origin xyz="0 0 0"/>
             <geometry>
                 <box size="0.05 0.05 0.05" />

File: src/myur5e/myur5e_description/urdf/mycamera.urdf.xacro (robot description, xacro)
@@ -33,5 +33,5 @@
     <xacro:property name="camera_link" value="0.02" /> <!-- Size of square 'camera' box -->
     <joint name="camera_joint" type="fixed">
-      <origin xyz="${wrist_length/2} 0 ${-wrist_radius-camera_link/2}" rpy="${pi} 0 0"/>
+      <origin xyz="${wrist_length/2} 0 ${wrist_radius+camera_link/2}" rpy="0 0 0"/>
       <parent link="wrist_attach"/>
       <child link="camera_link"/>

File: src/myur5e/myur5e_description/urdf/myur5e_robot.urdf.xacro (robot description, xacro)
@@ -26,4 +26,5 @@
   <xacro:include filename="$(find robotiq_85_description)/urdf/robotiq_85_gripper.urdf.xacro" />
   <!-- <xacro:include filename="$(find robotiq_description)/urdf/robotiq_85_gripper.urdf.xacro" /> -->
+  <!-- robotiq 85 -->
   <!--<xacro:include filename="$(find robotiq_2f_85_gripper_visualization)/urdf/robotiq_arg2f_85_model.xacro" />-->
   <!-- gripper -->
@@ -57,5 +58,5 @@
     <parent link="mytable"/>
     <child link="overcamera_link"/>
-    <origin xyz="0.75 0.0 1" rpy="${pi} ${3*pi/4} 0"/>
+    <origin xyz="0.75 0.0 0.8" rpy="${pi} ${3*pi/4} 0"/>
   </joint>
 </robot>

File: src/robotiq_85_gripper/robotiq_85_description/urdf/robotiq_85_gripper.transmission.xacro (robot description, xacro)
@@ -23,6 +23,6 @@
                 <joint>${prefix}gripper_finger1_joint</joint>
                 <mimicJoint>${prefix}gripper_finger2_inner_knuckle_joint</mimicJoint>
-                <!--multiplier>1.0</multiplier>
-                <offset>0.0</offset-->
+                <!-- <multiplier>-1.0</multiplier> -->
+                <!-- <offset>0.0</offset-->
             </plugin>
             <plugin filename="libroboticsgroup_gazebo_mimic_joint_plugin.so" name="${prefix}mimic_robotiq_85_3">

File: src/robotiq_85_gripper/robotiq_85_description/urdf/robotiq_85_gripper.urdf.xacro (robot description, xacro)
@@ -33,4 +33,5 @@
             <kp>100000000.0</kp>
             <kd>1.0</kd>
+            <turnGravityOff>1</turnGravityOff>
         </gazebo>
         <joint name="${prefix}gripper_finger1_joint" type="revolute">
@@ -74,4 +75,5 @@
             <kp>100000000.0</kp>
             <kd>1.0</kd>
+            <turnGravityOff>1</turnGravityOff>
         </gazebo>
         <link name="${prefix}gripper_finger2_knuckle_link">
@@ -100,4 +102,5 @@
             <kp>100000000.0</kp>
             <kd>1.0</kd>
+            <turnGravityOff>1</turnGravityOff>
         </gazebo>
         <joint name="${prefix}gripper_finger1_finger_joint" type="fixed">
@@ -136,4 +139,5 @@
             <kp>100000000.0</kp>
             <kd>1.0</kd>
+            <turnGravityOff>1</turnGravityOff>
         </gazebo>
         <link name="${prefix}gripper_finger2_finger_link">
@@ -162,4 +166,5 @@
             <kp>100000000.0</kp>
             <kd>1.0</kd>
+            <turnGravityOff>1</turnGravityOff>
         </gazebo>
         <joint name="${prefix}gripper_finger1_inner_knuckle_joint" type="continuous">
@@ -204,4 +209,5 @@
             <kp>100000000.0</kp>
             <kd>1.0</kd>
+            <turnGravityOff>1</turnGravityOff>
         </gazebo>
         <link name="${prefix}gripper_finger2_inner_knuckle_link">
@@ -230,4 +236,5 @@
             <kp>100000000.0</kp>
             <kd>1.0</kd>
+            <turnGravityOff>1</turnGravityOff>
         </gazebo>
         <joint name="${prefix}gripper_finger1_finger_tip_joint" type="continuous">
@@ -272,4 +279,5 @@
             <kp>100000000.0</kp>
             <kd>1.0</kd>
+            <turnGravityOff>1</turnGravityOff>
         </gazebo>
         <link name="${prefix}gripper_finger2_finger_tip_link">
@@ -298,4 +306,5 @@
             <kp>100000000.0</kp>
             <kd>1.0</kd>
+            <turnGravityOff>1</turnGravityOff>
         </gazebo>
 	<gazebo>
