Commit message: grasp plg fix

File: src/myur5e/myur5e_description/urdf/gzplugin_grasp_fix.urdf.xacro (robot description, xacro)
@@ -5,18 +5,18 @@
 		<gazebo>
 			<plugin name="gazebo_grasp_fix" filename="libgazebo_grasp_fix.so">
-					<arm>
-							<arm_name>myur5e_fix</arm_name>
-							<palm_link> gripper_finger1_inner_knuckle_link </palm_link>
-							<gripper_link>gripper_finger1_finger_tip_link</gripper_link>
-							<palm_link> gripper_finger2_inner_knuckle_link </palm_link>
-							<gripper_link>gripper_finger2_finger_tip_link</gripper_link>
-					</arm>
-					<forces_angle_tolerance>60</forces_angle_tolerance>
-					<update_rate>4</update_rate>
-					<grip_count_threshold>4</grip_count_threshold>
-					<max_grip_count>8</max_grip_count>
-					<release_tolerance>0.05</release_tolerance>
-					<disable_collisions_on_attach>true</disable_collisions_on_attach>
-					<contact_topic>__default_topic__</contact_topic>
+				<arm>
+					<arm_name>myur5e_fix</arm_name>
+					<palm_link> gripper_finger1_inner_knuckle_link </palm_link>
+					<gripper_link>gripper_finger1_finger_tip_link</gripper_link>
+					<palm_link> gripper_finger2_inner_knuckle_link </palm_link>
+					<gripper_link>gripper_finger2_finger_tip_link</gripper_link>
+				</arm>
+				<forces_angle_tolerance>100</forces_angle_tolerance>
+				<update_rate>4</update_rate>
+				<grip_count_threshold>4</grip_count_threshold>
+				<max_grip_count>8</max_grip_count>
+				<release_tolerance>0.005</release_tolerance>
+				<disable_collisions_on_attach>false</disable_collisions_on_attach>
+				<contact_topic>__default_topic__</contact_topic>
 			</plugin>
 		</gazebo>

File: src/myur5e/myur5e_description/urdf/mycamera.urdf.xacro (robot description, xacro)
@@ -24,5 +24,5 @@
     </link>
     <gazebo reference="wrist_attach">
-      <material>Gazebo/Green</material>
+      <material>Gazebo/FlatBlack</material>
     </gazebo>
     <joint name="wrist_joint" type="fixed">
@@ -50,5 +50,5 @@
           <box size="${camera_link} ${camera_link} ${camera_link}"/>
         </geometry>
-        <material name="red"/>
+        <!-- <material name="red"/> -->
       </visual>
       <inertial>
@@ -60,5 +60,5 @@
     <!-- camera -->
     <gazebo reference="camera_link">
-      <material>Gazebo/Red</material>
+      <material>Gazebo/RedTransparent</material>
       <sensor type="camera" name="wrist_camera">
         <update_rate>20.0</update_rate>

File: src/myur5e/myur5e_description/urdf/objects/mybox.urdf.xacro (robot description, xacro)
@@ -5,5 +5,5 @@
             <origin xyz="0 0 0" />
             <mass value="0.2" />
-            <inertia  ixx="1.0" ixy="0.0"  ixz="0.0"  iyy="100.0"  iyz="0.0"  izz="1.0" />
+            <inertia  ixx="1.0" ixy="1.0"  ixz="1.0"  iyy="1.0"  iyz="1.0"  izz="1.0" />
         </inertial>
         <visual>

Commit message: relocate

File: src/myur5e/myur5e_description/urdf/gzplugin_grasp_fix.urdf.xacro (robot description, xacro)
@@ -7,4 +7,5 @@
 				<arm>
 					<arm_name>myur5e_fix</arm_name>
+					<!-- <palm_link>wrist_3_link</palm_link> -->
 					<palm_link> gripper_finger1_inner_knuckle_link </palm_link>
 					<gripper_link>gripper_finger1_finger_tip_link</gripper_link>
@@ -16,5 +17,5 @@
 				<grip_count_threshold>4</grip_count_threshold>
 				<max_grip_count>8</max_grip_count>
-				<release_tolerance>0.005</release_tolerance>
+				<release_tolerance>0.03</release_tolerance>
 				<disable_collisions_on_attach>false</disable_collisions_on_attach>
 				<contact_topic>__default_topic__</contact_topic>

File: src/myur5e/myur5e_description/urdf/objects/mybox.urdf.xacro (robot description, xacro)
@@ -4,11 +4,11 @@
         <inertial>
             <origin xyz="0 0 0" />
-            <mass value="0.2" />
-            <inertia  ixx="1.0" ixy="1.0"  ixz="1.0"  iyy="1.0"  iyz="1.0"  izz="1.0" />
+            <mass value="0.3" />
+        <inertia  ixx="0.00003375" ixy="0.0"  ixz="0.0"  iyy="0.00003375"  iyz="0.0"  izz="0.00003375" />
         </inertial>
         <visual>
             <origin xyz="0 0 0"/>
             <geometry>
-                <box size="0.05 0.05 0.05" />
+                <box size="0.045 0.045 0.045" />
             </geometry>
         </visual>
@@ -16,10 +16,12 @@
             <origin xyz="0 0 0"/>
             <geometry>
-                <box size="0.05 0.05 0.05" />
+                <box size="0.045 0.045 0.045" />
             </geometry>
         </collision>
     </link>
     <gazebo reference="mybox">
-        <material>Gazebo/Blue</material>
+        <material>Gazebo/WoodPallet</material>
+        <mu1>1000</mu1>
+        <mu2>1000</mu2>
     </gazebo>
 </robot>

Commit message: add pid

File: src/myur5e/myur5e_description/urdf/gzplugin_grasp_fix.urdf.xacro (robot description, xacro)
@@ -13,5 +13,5 @@
 					<gripper_link>gripper_finger2_finger_tip_link</gripper_link>
 				</arm>
-				<forces_angle_tolerance>60</forces_angle_tolerance>
+				<forces_angle_tolerance>90</forces_angle_tolerance>
 				<update_rate>4</update_rate>
 				<grip_count_threshold>4</grip_count_threshold>

File: src/myur5e/myur5e_description/urdf/objects/mybox.urdf.xacro (robot description, xacro)
@@ -4,6 +4,6 @@
         <inertial>
             <origin xyz="0 0 0" />
-            <mass value="0.3" />
-        <inertia  ixx="0.00003375" ixy="0.0"  ixz="0.0"  iyy="0.00003375"  iyz="0.0"  izz="0.00003375" />
+            <mass value="0.2" />
+        <inertia  ixx="0.1" ixy="0.1"  ixz="0.1"  iyy="0.1"  iyz="0.1"  izz="0.1" />
         </inertial>
         <visual>
@@ -22,6 +22,6 @@
     <gazebo reference="mybox">
         <material>Gazebo/WoodPallet</material>
-        <mu1>1000</mu1>
-        <mu2>1000</mu2>
+        <mu1>0.5</mu1>
+        <mu2>0.4</mu2>
     </gazebo>
 </robot>

Commit message: small fix

File: src/myur5e/myur5e_description/urdf/gzplugin_grasp_fix.urdf.xacro (robot description, xacro)
@@ -16,5 +16,5 @@
 				<update_rate>10</update_rate>
 				<grip_count_threshold>1</grip_count_threshold>
-				<max_grip_count>5</max_grip_count>
+				<max_grip_count>3</max_grip_count>
 				<release_tolerance>0.01</release_tolerance>
 				<disable_collisions_on_attach>false</disable_collisions_on_attach>

File: src/myur5e/myur5e_description/urdf/objects/mycyl.urdf.xacro (robot description, xacro)
@@ -10,5 +10,5 @@
             <origin xyz="0 0 0"/>
             <geometry>
-                <cylinder radius="0.03" length="0.1"/>
+                <cylinder radius="0.03" length="0.05"/>
             </geometry>
         </visual>
@@ -16,10 +16,10 @@
             <origin xyz="0 0 0"/>
             <geometry>
-                <cylinder radius="0.03" length="0.1"/>
+                <cylinder radius="0.03" length="0.05"/>
             </geometry>
         </collision>
     </link>
-    <gazebo reference="mybox">
-        <material>Gazebo/Blue</material>
+    <gazebo reference="mycyl">
+        <material>Gazebo/Gold</material>
         <mu1>0.4</mu1>
         <mu2>0.3</mu2>
