Commit message: gym ready

File: src/myur5e/myur5e_description/urdf/mytable.urdf.xacro (robot description, xacro)
@@ -7,5 +7,5 @@
     <!-- rosrun gazebo_ros spawn_model -file $(rospack find ur5_single_arm_tufts)/urdf/objects/table.urdf -urdf -x 0.5 -y -0 -z 0.75 -model table -->
     <inertial>
-      <origin xyz="0.23 0 0.755" rpy="0 0 0" />
+      <origin xyz="0 0 0" rpy="0 0 0" />
       <mass value="1"/>
       <inertia
@@ -15,4 +15,5 @@
     </inertial>
     <visual>
+      <origin xyz="0 0 0" rpy="0 0 0" />
       <geometry>
         <box size="${table_xlength} ${table_ylength} ${table_zlength}"/>
@@ -20,4 +21,5 @@
     </visual>
     <collision>
+      <origin xyz="0 0 0" rpy="0 0 0" />
       <geometry>
         <box size="${table_xlength} ${table_ylength} ${table_zlength}"/>

File: src/myur5e/myur5e_description/urdf/myur5e_robot.urdf.xacro (robot description, xacro)
@@ -4,9 +4,8 @@
   <xacro:include filename="$(find ur_e_description)/urdf/common.gazebo.xacro" />
   <!-- ur5e -->
-  <!-- <xacro:include filename="$(find ur_e_description)/urdf/ur5e.urdf.xacro" /> -->
-  <!-- arm -->
+  <xacro:include filename="$(find ur_e_description)/urdf/ur5e.urdf.xacro" />
+  <!-- Unlimited -->
   <!-- <xacro:ur5e_robot prefix="" joint_limited="false"/> -->
   <!-- Limited -->
-  <xacro:include filename="$(find ur_e_description)/urdf/ur5e.urdf.xacro" />
   <xacro:ur5e_robot prefix="" joint_limited="true"
     shoulder_pan_lower_limit="${-pi}" shoulder_pan_upper_limit="${pi}"
@@ -17,16 +16,18 @@
     wrist_3_lower_limit="${-pi}" wrist_3_upper_limit="${pi}"
   />
+  <!-- robotiq 85 -->
+  <xacro:include filename="$(find robotiq_85_description)/urdf/robotiq_85_gripper.urdf.xacro" />
+  <!-- <xacro:include filename="$(find robotiq_description)/urdf/robotiq_85_gripper.urdf.xacro" /> -->
+  <!--<xacro:include filename="$(find robotiq_2f_85_gripper_visualization)/urdf/robotiq_arg2f_85_model.xacro" />-->
+  <!-- gripper without camera -->
+  <!-- <xacro:robotiq_85_gripper prefix="" parent="ee_link" >
+    <origin xyz="0 0 0" rpy="0 0 0"/>
+  </xacro:robotiq_85_gripper> -->
+  <!-- gripper with camera -->
   <!-- wrist camera -->
   <xacro:include filename="$(find myur5e_description)/urdf/mycamera.urdf.xacro" />
-  <!-- wrist camera attach -->
   <xacro:mywristcamera parent="ee_link" >
     <origin xyz="0 0 0" rpy="0 0 0"/>
   </xacro:mywristcamera>
-  <!-- robotiq 85 -->
-  <xacro:include filename="$(find robotiq_85_description)/urdf/robotiq_85_gripper.urdf.xacro" />
-  <!-- <xacro:include filename="$(find robotiq_description)/urdf/robotiq_85_gripper.urdf.xacro" /> -->
-  <!-- robotiq 85 -->
-  <!--<xacro:include filename="$(find robotiq_2f_85_gripper_visualization)/urdf/robotiq_arg2f_85_model.xacro" />-->
-  <!-- gripper -->
   <xacro:robotiq_85_gripper prefix="" parent="wrist_attach" >
     <origin xyz="${wrist_length} 0 0" rpy="0 0 0"/>
@@ -60,3 +61,5 @@
     <origin xyz="0.75 0.0 0.8" rpy="${pi} ${3*pi/4} 0"/>
   </joint>
+  <xacro:include filename="$(find myur5e_description)/urdf/gzplugin_grasp_fix.urdf.xacro"/>
+  <xacro:gzplugin_grasp_fix/>
 </robot>

Commit message: small fix

File: src/myur5e/myur5e_description/urdf/mytable.urdf.xacro (robot description, xacro)
@@ -1,6 +1,6 @@
 <?xml version="1.0"?>
 <robot xmlns:xacro="http://www.ros.org/wiki/xacro" name="mytable" >
-  <xacro:property name="table_xlength" value="1" />
-  <xacro:property name="table_ylength" value="1.5" />
+  <xacro:property name="table_xlength" value="1.2" />
+  <xacro:property name="table_ylength" value="2" />
   <xacro:property name="table_zlength" value="0.05" />
   <link name="mytable">
