Commit message: add conveyor

File: src/myur5e/myur5e_description/urdf/mypedestal.urdf.xacro (robot description, xacro)
@@ -2,5 +2,5 @@
 <robot xmlns:xacro="http://www.ros.org/wiki/xacro" name="mypedestal" >
   <xacro:property name="pe_radius" value="0.1" />
-  <xacro:property name="pedestal_height" value="1.0" />
+  <xacro:property name="pedestal_height" value="0.75" />
   <link name="mypedestal">
     <inertial>

File: src/myur5e/myur5e_description/urdf/objects/mybox.urdf.xacro (robot description, xacro)
@@ -4,5 +4,5 @@
         <inertial>
             <origin xyz="0 0 0" />
-            <mass value="0.05" />
+            <mass value="0.1" />
         <inertia  ixx="0.001" ixy="0"  ixz="0"  iyy="0.001"  iyz="0"  izz="0.001" />
         </inertial>

File: src/myur5e/myur5e_description/urdf/objects/mycyl.urdf.xacro (robot description, xacro)
@@ -4,5 +4,5 @@
         <inertial>
             <origin xyz="0 0 0" />
-            <mass value="0.05" />
+            <mass value="0.1" />
         <inertia  ixx="0.0001" ixy="0"  ixz="0"  iyy="0.0001"  iyz="0"  izz="0.0001" />
         </inertial>
@@ -21,5 +21,5 @@
     </link>
     <gazebo reference="mycyl">
-        <material>Gazebo/Gold</material>
+        <material>Gazebo/Green</material>
         <mu1>0.4</mu1>
         <mu2>0.3</mu2>

Commit message: update real height of pedestal and table

File: src/myur5e/myur5e_description/urdf/mypedestal.urdf.xacro (robot description, xacro)
@@ -2,5 +2,5 @@
 <robot xmlns:xacro="http://www.ros.org/wiki/xacro" name="mypedestal" >
   <xacro:property name="pe_radius" value="0.1" />
-  <xacro:property name="pedestal_height" value="0.75" />
+  <xacro:property name="pedestal_height" value="0.95" />
   <link name="mypedestal">
     <inertial>

File: src/myur5e/myur5e_description/urdf/myur5e_robot.urdf.xacro (robot description, xacro)
@@ -40,5 +40,5 @@
   <xacro:include filename="$(find myur5e_description)/urdf/my_overview_camera.urdf.xacro" />
   <link name="world" />
-  <xacro:property name="table_height" value="0.95" />
+  <xacro:property name="table_height" value="0.7" />
   <joint name="world_joint" type="fixed">
     <parent link="world" />
@@ -49,5 +49,5 @@
     <parent link="world"/>
     <child link="mytable"/>
-    <origin xyz="0.61 0.0 ${table_height}" rpy="0 0 0"/>
+    <origin xyz="0.7 0.0 ${table_height}" rpy="0 0 0"/>
   </joint>
   <joint name="robot_to_pedestal" type="fixed">
