Commit message: small fix table

File: src/myur5e/myur5e_description/urdf/myur5e_robot.urdf.xacro (robot description, xacro)
@@ -49,5 +49,5 @@
     <parent link="world"/>
     <child link="mytable"/>
-    <origin xyz="0.8 0.0 ${table_height}" rpy="0 0 0"/>
+    <origin xyz="0.61 0.0 ${table_height}" rpy="0 0 0"/>
   </joint>
   <joint name="robot_to_pedestal" type="fixed">

Commit message: phase 2 dev, using world file gazebo

File: src/myur5e/myur5e_description/urdf/myur5e_robot.urdf.xacro (robot description, xacro)
@@ -34,7 +34,7 @@
   </xacro:robotiq_85_gripper>
   <!-- pedestal -->
-  <xacro:include filename="$(find myur5e_description)/urdf/mypedestal.urdf.xacro" />
+  <xacro:include filename="$(find myur5e_description)/urdf/objects/mypedestal.urdf.xacro" />
   <!-- table -->
-  <xacro:include filename="$(find myur5e_description)/urdf/mytable.urdf.xacro" />
+  <xacro:include filename="$(find myur5e_description)/urdf/objects/mytable.urdf.xacro" />
   <!-- overview camera -->
   <xacro:include filename="$(find myur5e_description)/urdf/my_overview_camera.urdf.xacro" />

File: src/myur5e/myur5e_description/urdf/myur5e_robot_without_table.urdf.xacro (robot description, xacro)
@@ -34,5 +34,5 @@
   </xacro:robotiq_85_gripper>
   <!-- pedestal -->
-  <xacro:include filename="$(find myur5e_description)/urdf/mypedestal.urdf.xacro" />
+  <xacro:include filename="$(find myur5e_description)/urdf/objects/mypedestal.urdf.xacro" />
   <link name="world" />
   <joint name="world_joint" type="fixed">

File: src/myur5e/myur5e_description/urdf/myur5e_with_gripper_for_moveit.urdf.xacro (robot description, xacro)
@@ -1,10 +1,19 @@
 <?xml version="1.0"?>
 <robot xmlns:xacro="http://www.ros.org/wiki/xacro" name="myur5e" >
+  <!-- common stuff -->
+  <xacro:include filename="$(find ur_e_description)/urdf/common.gazebo.xacro" />
   <!-- ur5e -->
   <xacro:include filename="$(find ur_e_description)/urdf/ur5e.urdf.xacro" />
-  <!-- arm -->
-  <xacro:ur5e_robot prefix="" joint_limited="false"/>
-  <!-- robotiq 85 -->
-  <!--<xacro:include filename="$(find robotiq_2f_85_gripper_visualization)/urdf/robotiq_arg2f_85_model.xacro" />-->
+  <!-- Unlimited -->
+  <!-- <xacro:ur5e_robot prefix="" joint_limited="false"/> -->
+  <!-- Limited -->
+  <xacro:ur5e_robot prefix="" joint_limited="true"
+    shoulder_pan_lower_limit="${-pi}" shoulder_pan_upper_limit="${pi}"
+    shoulder_lift_lower_limit="${-pi}" shoulder_lift_upper_limit="${pi}"
+    elbow_joint_lower_limit="${-pi}" elbow_joint_upper_limit="${pi}"
+    wrist_1_lower_limit="${-pi}" wrist_1_upper_limit="${pi}"
+    wrist_2_lower_limit="${-pi}" wrist_2_upper_limit="${pi}"
+    wrist_3_lower_limit="${-pi}" wrist_3_upper_limit="${pi}"
+  />
   <!-- wrist camera -->
   <xacro:include filename="$(find myur5e_description)/urdf/mycamera.urdf.xacro" />
@@ -22,6 +31,8 @@
   <joint name="world_joint" type="fixed">
     <parent link="world" />
-    <child link="base_link" /> <!-- TODO: check base_link name of robot -->
+    <child link="base_link" />
     <origin xyz="0.0 0.0 0.0" rpy="0.0 0.0 0.0" />
   </joint>
+  <xacro:include filename="$(find myur5e_description)/urdf/gzplugin_grasp_fix.urdf.xacro"/>
+  <xacro:gzplugin_grasp_fix/>
 </robot>
