Commit message: work fine

File: src/myur5e/myur5e_description/urdf/mycamera.urdf.xacro (robot description, xacro)
@@ -33,5 +33,5 @@
     <xacro:property name="camera_link" value="0.02" /> <!-- Size of square 'camera' box -->
     <joint name="camera_joint" type="fixed">
-      <origin xyz="${wrist_length/2} 0 ${-wrist_radius-camera_link/2}" rpy="0 0 0"/>
+      <origin xyz="${wrist_length/2} 0 ${-wrist_radius-camera_link/2}" rpy="${pi} 0 0"/>
       <parent link="wrist_attach"/>
       <child link="camera_link"/>
@@ -71,6 +71,6 @@
           </image>
           <clip>
-            <near>0.02</near>
-            <far>300</far>
+            <near>0.01</near>
+            <far>10</far>
           </clip>
           <noise>

File: src/myur5e/myur5e_description/urdf/myur5e_robot.urdf.xacro (robot description, xacro)
@@ -17,4 +17,5 @@
   <!-- robotiq 85 -->
   <xacro:include filename="$(find robotiq_85_description)/urdf/robotiq_85_gripper.urdf.xacro" />
+  <!-- <xacro:include filename="$(find robotiq_description)/urdf/robotiq_85_gripper.urdf.xacro" /> -->
   <!-- gripper -->
   <xacro:robotiq_85_gripper prefix="" parent="wrist_attach" >
@@ -47,5 +48,5 @@
     <parent link="mytable"/>
     <child link="overcamera_link"/>
-    <origin xyz="0.0 0.0 1" rpy="0 ${pi/2} 0"/>
+    <origin xyz="0.75 0.0 1" rpy="${pi} ${3*pi/4} 0"/>
   </joint>
 </robot>

Commit message: match sim with real size

File: src/myur5e/myur5e_description/urdf/mycamera.urdf.xacro (robot description, xacro)
@@ -64,8 +64,8 @@
         <update_rate>20.0</update_rate>
         <camera name="wrist_cam">
-          <horizontal_fov>1.3962634</horizontal_fov>
+          <horizontal_fov>0.69</horizontal_fov>
           <image>
-            <width>512</width>
-            <height>512</height>
+            <width>640</width>
+            <height>480</height>
             <format>R8G8B8</format>
           </image>

File: src/myur5e/myur5e_description/urdf/mytable.urdf.xacro (robot description, xacro)
@@ -28,5 +28,5 @@
   </link>
   <gazebo reference="mytable">
-    <material>Gazebo/Wood</material>
+    <material>Gazebo/DarkGrey</material>
     <static>True</static>
   </gazebo>

File: src/myur5e/myur5e_description/urdf/myur5e_robot.urdf.xacro (robot description, xacro)
@@ -59,5 +59,5 @@
     <parent link="mytable"/>
     <child link="overcamera_link"/>
-    <origin xyz="0.75 0.0 0.8" rpy="${pi} ${3*pi/4} 0"/>
+    <origin xyz="0.6 0.0 0.3" rpy="${pi} ${4*pi/5} 0"/>
   </joint>
   <xacro:include filename="$(find myur5e_description)/urdf/gzplugin_grasp_fix.urdf.xacro"/>

Commit message: world complete

File: src/myur5e/myur5e_description/urdf/mycamera.urdf.xacro (robot description, xacro)
@@ -2,5 +2,5 @@
 <robot xmlns:xacro="http://www.ros.org/wiki/xacro" name="mywristcamera" >
   <xacro:property name="wrist_radius" value="0.04" />
-  <xacro:property name="wrist_length" value="0.02" />
+  <xacro:property name="wrist_length" value="0.01" />
   <xacro:macro name="mywristcamera" params="parent *origin">
     <link name="wrist_attach">
@@ -33,5 +33,5 @@
     <xacro:property name="camera_link" value="0.02" /> <!-- Size of square 'camera' box -->
     <joint name="camera_joint" type="fixed">
-      <origin xyz="${wrist_length/2} 0 ${wrist_radius+camera_link/2}" rpy="0 0 0"/>
+      <origin xyz="${wrist_length/2} 0 ${-wrist_radius-camera_link/2}" rpy="0 0 0"/>
       <parent link="wrist_attach"/>
       <child link="camera_link"/>
