Commit message: relocate

File: src/myur5e/myur5e_description/urdf/objects/mybox.urdf.xacro (robot description, xacro)
@@ -10,5 +10,5 @@
             <origin xyz="0 0 0"/>
             <geometry>
-                <box size="0.045 0.045 0.045" />
+                <box size="0.045 0.045 0.1" />
             </geometry>
         </visual>
@@ -16,5 +16,5 @@
             <origin xyz="0 0 0"/>
             <geometry>
-                <box size="0.045 0.045 0.045" />
+                <box size="0.045 0.045 0.1" />
             </geometry>
         </collision>

Commit message: small fix

File: src/myur5e/myur5e_description/urdf/objects/mybox.urdf.xacro (robot description, xacro)
@@ -4,6 +4,6 @@
         <inertial>
             <origin xyz="0 0 0" />
-            <mass value="0.2" />
-        <inertia  ixx="0.1" ixy="0.1"  ixz="0.1"  iyy="0.1"  iyz="0.1"  izz="0.1" />
+            <mass value="0.05" />
+        <inertia  ixx="0.001" ixy="0"  ixz="0"  iyy="0.001"  iyz="0"  izz="0.001" />
         </inertial>
         <visual>
@@ -21,7 +21,9 @@
     </link>
     <gazebo reference="mybox">
-        <material>Gazebo/WoodPallet</material>
-        <mu1>0.5</mu1>
-        <mu2>0.4</mu2>
+        <material>Gazebo/Blue</material>
+        <mu1>0.4</mu1>
+        <mu2>0.3</mu2>
+        <kp>10000</kp>
+        <kd>1</kd>
     </gazebo>
 </robot>

Commit message: small fix pickplace worked

File: src/myur5e/myur5e_description/urdf/objects/mybox.urdf.xacro (robot description, xacro)
@@ -10,5 +10,5 @@
             <origin xyz="0 0 0"/>
             <geometry>
-                <box size="0.045 0.045 0.1" />
+                <box size="0.05 0.05 0.05" />
             </geometry>
         </visual>
@@ -16,5 +16,5 @@
             <origin xyz="0 0 0"/>
             <geometry>
-                <box size="0.045 0.045 0.1" />
+                <box size="0.05 0.05 0.05" />
             </geometry>
         </collision>

File: src/myur5e/myur5e_description/urdf/objects/mycyl.urdf.xacro (robot description, xacro)
@@ -10,5 +10,5 @@
             <origin xyz="0 0 0"/>
             <geometry>
-                <cylinder radius="0.03" length="0.05"/>
+                <cylinder radius="0.025" length="0.05"/>
             </geometry>
         </visual>
@@ -16,5 +16,5 @@
             <origin xyz="0 0 0"/>
             <geometry>
-                <cylinder radius="0.03" length="0.05"/>
+                <cylinder radius="0.025" length="0.05"/>
             </geometry>
         </collision>
