Commit message: conveyor added

File: src/myur5e/myur5e_description/urdf/conveyor/simple_conveyor.urdf.xacro (robot description, xacro)
@@ -33,8 +33,8 @@
 	</link>
 	<gazebo reference="belt_visual">
-        <material>Gazebo/White</material>
+        <material>Gazebo/DarkGrey</material>
     </gazebo>
 	<joint name="belt_joint" type="prismatic">
-		<origin xyz="0.0 0.0 0.025" rpy="0.0 0.0 0.0"/>
+		<origin xyz="0.0 -0.3 0.025" rpy="0.0 0.0 0.0"/>
 		<parent link="belt_visual"/>
 		<child link="belt_moving"/>
@@ -48,20 +48,20 @@
 			<inertia ixx="0.0" ixy="0.0" ixz="0.0" iyy="0.0" iyz="0.0" izz="0.0"/>
 		</inertial>
-		<visual>
+		<!-- <visual>
 			<origin xyz="0.0 0.0 0.0005" rpy="0.0 0.0 0.0"/>
 			<geometry>
-				<box size="0.2 1.5 0.001"/>
+				<box size="0.2 1.8 0.001"/>
 			</geometry>
-		</visual>
+		</visual> -->
 		<collision>
 			<origin xyz="0.0 0.0 0.0005" rpy="0.0 0.0 0.0"/>
 			<geometry>
-				<box size="0.2 1.5 0.001"/>
+				<box size="0.2 1.8 0.001"/>
 			</geometry>
 		</collision>
 	</link>
-	<gazebo reference="belt_moving">
-        <material>Gazebo/DarkGrey</material>
-    </gazebo>
+	<!-- <gazebo reference="belt_moving">
+        <material>Gazebo/Grey</material>
+    </gazebo> -->
 	<gazebo>
 		<plugin name="conveyor_belt_plugin" filename="libROSConveyorBeltPlugin.so">
